File: base-controller/base-controller.kicad_sch (KiCad schematic)
At the start: 59 parts, among them J1 24V_IN, J2 MOTOR_CONTROL, J3 LIMIT_A, J4 LIMIT_B, J5 SPARE_IO, J6 XIAO_POWER_LINK, J7 MOTOR_24V_OUT, Q1 MMBT3904, Q2 MMBT3904, Q3 MMBT3904, SW1 XUNPU TS-1088-AR02016, U1 XIAO-ESP32-C6, U2 LMR51420XDDCR, U3 TPS26600PWP

Commit message: Save JLC assembly placement corrections and export guidance
Parts:
- C7, J2, J3, J4: FT Rotation Offset (none) -> 180
- J1, J7: FT Position Offset (none) -> 0,-0.7925; FT Rotation Offset (none) -> 180
- J5, J6, U2: FT Rotation Offset (none) -> 90
- SW1: LCSC (none) -> C720477; MPN C720477 -> TS-1088-AR02016; Manufacturer (none) -> XUNPU
- U3: FT Rotation Offset (none) -> -90; LCSC (none) -> C544399; MPN (none) -> TPS26600PWPR; Manufacturer (none) -> Texas Instruments
Changed lines of the file:
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@@
 			)
 		)
+		(property "FT Rotation Offset" "90"
+			(at 283.21 39.37 0)
+			(effects
+				(font
+					(size 1.27 1.27)
+				)
+				(hide yes)
+			)
+		)
 		(pin "6"
 		)
@@
 			)
 		)
+		(property "FT Rotation Offset" "180"
+			(at 67.31 36.83 0)
+			(effects
+				(font
+					(size 1.27 1.27)
+				)
+				(hide yes)
+			)
+		)
+		(property "FT Position Offset" "0,-0.7925"
+			(at 67.31 36.83 0)
+			(effects
+				(font
+					(size 1.27 1.27)
+				)
+				(hide yes)
+			)
+		)
 		(pin "2"
 		)
@@
 			)
 		)
+		(property "FT Rotation Offset" "90"
+			(at 265.43 175.26 0)
+			(effects
+				(font
+					(size 1.27 1.27)
+				)
+				(hide yes)
+			)
+		)
 		(pin "2"
 		)
@@
 			)
 		)
+		(property "FT Rotation Offset" "180"
+			(at 134.62 245.11 0)
+			(effects
+				(font
+					(size 1.27 1.27)
+				)
+				(hide yes)
+			)
+		)
 		(pin "1"
 		)
@@
 			)
 		)
+		(property "FT Rotation Offset" "180"
+			(at 78.74 245.11 0)
+			(effects
+				(font
+					(size 1.27 1.27)
+				)
+				(hide yes)
+			)
+		)
 		(pin "1"
 		)
@@
 			)
 		)
+		(property "FT Rotation Offset" "180"
+			(at 218.44 44.45 0)
+			(effects
+				(font
+					(size 1.27 1.27)
+				)
+				(hide yes)
+			)
+		)
 		(pin "2"
 		)
@@
 			)
 		)
+		(property "FT Rotation Offset" "180"
+			(at 125.73 133.35 0)
+			(effects
+				(font
+					(size 1.27 1.27)
+				)
+				(hide yes)
+			)
+		)
 		(pin "1"
 		)
@@
 			)
 		)
+		(property "Manufacturer" "Texas Instruments"
+			(at 140.97 49.53 0)
+			(effects
+				(font
+					(size 1.27 1.27)
+				)
+				(hide yes)
+			)
+		)
+		(property "MPN" "TPS26600PWPR"
+			(at 140.97 49.53 0)
+			(effects
+				(font
+					(size 1.27 1.27)
+				)
+				(hide yes)
+			)
+		)
+		(property "LCSC" "C544399"
+			(at 140.97 49.53 0)
+			(effects
+				(font
+					(size 1.27 1.27)
+				)
+				(hide yes)
+			)
+		)
+		(property "FT Rotation Offset" "-90"
+			(at 140.97 49.53 0)
+			(effects
+				(font
+					(size 1.27 1.27)
+				)
+				(hide yes)
+			)
+		)
 		(pin "17"
 		)
@@
 			)
 		)
-		(property "MPN" "C720477"
+		(property "MPN" "TS-1088-AR02016"
 			(at 203.2 250.19 0)
 			(effects
@@
 			)
 		)
+		(property "Manufacturer" "XUNPU"
+			(at 203.2 250.19 90)
+			(effects
+				(font
+					(size 1.27 1.27)
+				)
+				(hide yes)
+			)
+		)
+		(property "LCSC" "C720477"
+			(at 203.2 250.19 90)
+			(effects
+				(font
+					(size 1.27 1.27)
+				)
+				(hide yes)
+			)
+		)
 		(pin "2"
 		)
@@
 			)
 		)
+		(property "FT Rotation Offset" "180"
+			(at 68.58 72.39 0)
+			(effects
+				(font
+					(size 1.27 1.27)
+				)
+				(hide yes)
+			)
+		)
+		(property "FT Position Offset" "0,-0.7925"
+			(at 68.58 72.39 0)
+			(effects
+				(font
+					(size 1.27 1.27)
+				)
+				(hide yes)
+			)
+		)
 		(pin "2"
 		)
@@
 			(at 205.74 168.91 0)
 			(effects
+				(font
+					(size 1.27 1.27)
+				)
+				(hide yes)
+			)
+		)
+		(property "FT Rotation Offset" "90"
+			(at 205.74 168.91 0)
+			(effects
